File: pcb/pcb.kicad_sch (KiCad schematic)
At the start: 28 parts, among them J1 Conn_01x02, J2 Conn_01x02, SW1 SW_SPDT, U1 TL072, U3 AP63205WU

Commit message: pcb v1
Parts:
- added H1, H2, H3, H4: MountingHole_Pad, MountingHole:MountingHole_2.2mm_M2, symbol Mechanical:MountingHole_Pad

Commit message: pcb v2: distortion stage
Parts:
- added D1, D2: 1N4148, symbol Device:D_Small
- added RV2: 100k, symbol Device:R_Potentiometer
- R6: value 47 -> 4k7; footprint Resistor_SMD:R_0402_1005Metric -> (none)
- RV1: value R_Potentiometer -> 10k
Connections:
- net GND: now also R6.1, RV2.1; no longer R6.2, RV1.1, RV1.3
- net GNDPWR: now also RV1.1
- net at U1.5 (+): now also C2.2, R5.1
- net at U1.6 (-): now also R6.2, D1.1 (K), D2.2 (A)
- net at U1.7: now also RV1.3, RV2.3
- new net: D1.2 (A), D2.1 (K), RV2.2
Other:
- moved on the sheet: C7, C8, H1, H2, H3, H4, RV1, U1B, U2
